Commit message: refactor:重写源代码函数命名问题

File: drop_point_prediction/src/volleyball_robot_description/urdf/volleyball_robot_description.urdf.xacro (robot description, xacro)
@@ -19,8 +19,4 @@
                 xyz="0 0 0"
                 rpy="0 0 0" />
-            <geometry>
-                <mesh
-                filename="package://volleyball_robot_description/meshes/base_link.STL" />
-            </geometry>
             <material
                 name="">
@@ -35,8 +31,4 @@
                 xyz="0 0 0"
                 rpy="0 0.5841617 0" />
-            <geometry>
-                <mesh
-                filename="package://volleyball_robot_description/meshes/delta_arm_link.STL" />
-            </geometry>
             <material
                 name="">
@@ -60,8 +52,4 @@
                 xyz="0 0 0"
                 rpy="0 0 0" />
-            <geometry>
-                <mesh
-                filename="package://volleyball_robot_description/meshes/camera_link.STL" />
-            </geometry>
             <material
                 name="">
